File: PCB/Working - Under Develolpment/Index Registers 1.1/Index Registers - 1.1.sch (EAGLE design)
At the start: 83 parts, among them IC1 74LS32N, IC10 74LS32N, IC11 74LS192N, IC12 74LS192N, IC13 74LS192N, IC14 74LS192N, IC15 74LS244N, IC16 74LS244N, IC17 74LS32N, IC18 74LS192N, IC19 74LS192N, IC2 74LS32N, IC20 74LS192N, IC21 74LS192N, IC22 74LS244N, IC23 74LS244N, IC24 74LS32N, IC25 74LS192N, IC26 74LS192N, IC27 74LS192N, IC28 74LS192N, IC29 74LS244N, IC3 74LS192N, IC30 74LS244N, IC31 74LS32N, IC32 74LS139N, IC33 74LS139N, IC34 4077N, IC35 74LS245N, IC36 74LS245N, IC37 74LS245N, IC4 74LS192N, IC5 74LS192N, IC6 74LS192N, IC7 74LS244N, IC8 74LS244N, IC9 74LS32N, X1 FABC96R

Commit message: Index Register Board V1.1
Modify so any data register can drive address bus
Parts:
- removed IC16: 74LS244N, 74xx-us:74LS244N
- removed JP1, JP2: (no value), pinhead:PINHD-2X20
- added IC38: 74LS139N, 74xx-us:74LS139N
- added IC40, IC47: 74LS32N, 74xx-us:74LS32N
- added IC41, IC42, IC45, IC46, IC49, IC50: 74LS244N, 74xx-us:74LS244N
- added IC43, IC44: 74LS192N, 74xx-us:74LS192N
- added J3: (no value), SparkFun-Connectors:M04X2
- IC10, IC9: value 74LS32N -> 74LS192N; device 74xx-us:74LS32N -> 74xx-us:74LS192N
- IC13, IC14, IC18, IC27, IC28: value 74LS192N -> 74LS244N; device 74xx-us:74LS192N -> 74xx-us:74LS244N
- IC15: value 74LS244N -> 74LS32N; device 74xx-us:74LS244N -> 74xx-us:74LS32N
- IC17, IC24: value 74LS32N -> 74LS244N; device 74xx-us:74LS32N -> 74xx-us:74LS244N
- IC22, IC29, IC30: value 74LS244N -> 74LS192N; device 74xx-us:74LS244N -> 74xx-us:74LS192N
- IC25, IC26: value 74LS192N -> 74LS32N; device 74xx-us:74LS192N -> 74xx-us:74LS32N
Connections:
- net IO-ADDR0 renamed IOADDR0
- net IO-ADDR1 renamed IOADDR1
- net IO-ADDR2 renamed IOADDR2
- net IO-ADDR3 renamed IOADDR3
- removed net -ADDR-REG-LD0: X1-C4.B
- removed net -ADDR-REG-LD1: X1-C6.B
- removed net -ADDR-REG-RD0: X1-C3.B
- removed net -ADDR-REG-RD1: X1-C5.B
- removed net 1C-12: JP1.29
- removed net IA-0: IC11A.QA, IC15B.A1, JP2.5
- removed net IA-1: IC11A.QB, IC15B.A2, JP2.7
- removed net IA-10: IC13A.QC, IC16B.A3, JP2.25
- removed net IA-11: IC13A.QD, IC16B.A4, JP2.27
- removed net IA-12: IC14A.QA, IC16A.A1, JP2.29
- removed net IA-13: IC14A.QB, IC16A.A2, JP2.31
- removed net IA-14: IC14A.QC, IC16A.A3, JP2.33
- removed net IA-15: IC14A.QD, IC16A.A4, JP2.35
- removed net IA-2: IC11A.QC, IC15B.A3, JP2.9
- removed net IA-3: IC11A.QD, IC15B.A4, JP2.11
- removed net IA-4: IC12A.QA, IC15A.A1, JP2.13
- removed net IA-5: IC12A.QB, IC15A.A2, JP2.15
- removed net IA-6: IC12A.QC, IC15A.A3, JP2.17
- removed net IA-7: IC12A.QD, IC15A.A4, JP2.19
- removed net IA-8: IC13A.QA, IC16B.A1, JP2.21
- removed net IA-9: IC13A.QB, IC16B.A2, JP2.23
- removed net IB-0: JP2.6
- removed net IB-1: JP2.8
- removed net IB-10: JP2.26
- removed net IB-11: JP2.28
- removed net IB-12: JP2.30
- removed net IB-13: JP2.32
- removed net IB-14: JP2.34
- removed net IB-15: JP2.36
- removed net IB-2: JP2.10
- removed net IB-3: JP2.12
- removed net IB-4: JP2.14
- removed net IB-5: JP2.16
- removed net IB-6: JP2.18
- removed net IB-7: JP2.20
- removed net IB-8: JP2.22
- removed net IB-9: JP2.24
- removed net IC-0: IC25A.QA, IC29B.A1, JP1.5
- removed net IC-1: IC25A.QB, IC29B.A2, JP1.7
- removed net IC-10: IC27A.QC, IC30B.A3, JP1.25
- removed net IC-11: IC27A.QD, IC30B.A4, JP1.27
- removed net IC-12: IC28A.QA, IC30A.A1
- removed net IC-13: IC28A.QB, IC30A.A2, JP1.31
- removed net IC-14: IC28A.QC, IC30A.A3, JP1.33
- removed net IC-15: IC28A.QD, IC30A.A4, JP1.35
- removed net IC-2: IC25A.QC, IC29B.A3, JP1.9
- removed net IC-3: IC25A.QD, IC29B.A4, JP1.11
- removed net IC-4: IC26A.QA, IC29A.A1, JP1.13
- removed net IC-5: IC26A.QB, IC29A.A2, JP1.15
- removed net IC-6: IC26A.QC, IC29A.A3, JP1.17
- removed net IC-7: IC26A.QD, IC29A.A4, JP1.19
- removed net IC-8: IC27A.QA, IC30B.A1, JP1.21
- removed net IC-9: IC27A.QB, IC30B.A2, JP1.23
- removed net ID-0: JP1.6
- removed net ID-1: JP1.8
- removed net ID-10: JP1.26
- removed net ID-11: JP1.28
- removed net ID-12: JP1.30
- removed net ID-13: JP1.32
- removed net ID-14: JP1.34
- removed net ID-15: JP1.36
- removed net ID-2: JP1.10
- removed net ID-3: JP1.12
- removed net ID-4: JP1.14
- removed net ID-5: JP1.16
- removed net ID-6: JP1.18
- removed net ID-7: JP1.20
- removed net ID-8: JP1.22
- removed net ID-9: JP1.24
- removed net N$58 (its old number): IC18A.BO, IC19A.DN
- removed net N$59 (its old number): IC18A.CO, IC19A.UP
- removed net N$6 (its old number): IC27A.BO, IC28A.DN
- removed net N$7 (its old number): IC27A.CO, IC28A.UP
- removed net UNUSED0: X1-C12.B
- new net -ADDRSEL: IC38A.G, J3.2, J3.4, J3.6, J3.8
- new net -ARD0: IC38B.Y0, J3.1
- new net -R0-ADDRSEL: IC38A.Y0, IC41A.G, IC41B.G, IC42A.G, IC42B.G
- new net -R1-ADDRSEL: IC17A.G, IC17B.G, IC18A.G, IC18B.G, IC38A.Y1
- new net -R2-ADDRSEL: IC27A.G, IC27B.G, IC28A.G, IC28B.G, IC38A.Y2
- new net -R3-ADDRSEL: IC38A.Y3, IC49A.G, IC49B.G, IC50A.G, IC50B.G
- new net -VMA: IC40A.I1, X1-C12.B
- new net ADDR-REG-ID0: IC38A.A, X1-C3.B
- new net ADDR-REG-ID1: IC38A.B, X1-C4.B
- new net ADDR-REG-ID2: IC38B.A, X1-C5.B
- new net ADDR-REG-ID3: IC38B.B, X1-C6.B
- new net N$100: IC29A.QC, IC45B.A3, IC49A.A3
- new net N$101: IC29A.QD, IC45B.A4, IC49A.A4
- new net N$102: IC30A.QA, IC45A.A1, IC49B.A1
- new net N$103: IC30A.QB, IC45A.A2, IC49B.A2
- new net N$104: IC30A.QC, IC45A.A3, IC49B.A3
- new net N$105: IC30A.QD, IC45A.A4, IC49B.A4
- new net N$106: IC43A.QA, IC46B.A1, IC50A.A1
- new net N$107: IC43A.QB, IC46B.A2, IC50A.A2
- new net N$108: IC43A.QC, IC46B.A3, IC50A.A3
- new net N$109: IC43A.QD, IC46B.A4, IC50A.A4
- new net N$110: IC44A.QA, IC46A.A1, IC50B.A1
- new net N$111: IC44A.QB, IC46A.A2, IC50B.A2
- new net N$112: IC44A.QC, IC46A.A3, IC50B.A3
- new net N$113: IC44A.QD, IC46A.A4, IC50B.A4
- new net N$28: IC13B.A1, IC17A.A1, IC9A.QA
- new net N$29: IC13B.A2, IC17A.A2, IC9A.QB
- new net N$45: IC38B.G, IC40A.O
- new net N$51: IC38B.Y1, J3.3
- new net N$52: IC38B.Y2, J3.5
- new net N$53: IC38B.Y3, J3.7
- new net N$54: IC12A.QA, IC14A.A1, IC18B.A1
- new net N$55: IC12A.QB, IC14A.A2, IC18B.A2
- new net N$56: IC12A.QC, IC14A.A3, IC18B.A3
- new net N$57: IC12A.QD, IC14A.A4, IC18B.A4
- new net N$62: IC21A.BO, IC22A.DN
- new net N$63: IC21A.CO, IC22A.UP
- new net N$67: IC23A.G, IC23B.G, IC26A.O
- new net N$68: IC24A.G, IC24B.G, IC26B.O
- new net N$69: IC21A.LD, IC22A.LD, IC25D.O
- new net N$70: IC19A.QA, IC23B.A1, IC27A.A1
- new net N$71: IC19A.QB, IC23B.A2, IC27A.A2
- new net N$72: IC19A.QC, IC23B.A3, IC27A.A3
- new net N$73: IC19A.QD, IC23B.A4, IC27A.A4
- new net N$74: IC20A.QA, IC23A.A1, IC27B.A1
- new net N$75: IC20A.QB, IC23A.A2, IC27B.A2
- new net N$76: IC20A.QC, IC23A.A3, IC27B.A3
- new net N$77: IC20A.QD, IC23A.A4, IC27B.A4
- new net N$78: IC21A.QA, IC24B.A1, IC28A.A1
- new net N$79: IC21A.QB, IC24B.A2, IC28A.A2
- new net N$99: IC29A.QB, IC45B.A2, IC49A.A2
- net -BUS-EN: now also IC40A.I0
- net -R0-LDSEL: now also IC1C.I0, IC1D.I0; no longer IC9C.I0, IC9D.I0
- net -R0-RDSEL: now also IC1A.I0, IC1B.I0, IC2A.I0, IC2B.I0; no longer IC10A.I0, IC10B.I0, IC9A.I0, IC9B.I0
- net -R1-LDSEL: now also IC15C.I0, IC15D.I0; no longer IC24C.I0, IC24D.I0
- net -R1-RDSEL: now also IC15A.I0, IC15B.I0, IC2C.I0, IC2D.I0; no longer IC10C.I0, IC10D.I0, IC24A.I0, IC24B.I0
- net -R2-LDSEL: now also IC25C.I0, IC25D.I0; no longer IC1C.I0, IC1D.I0
- net -R2-RDSEL: now also IC25A.I0, IC25B.I0, IC26A.I0, IC26B.I0; no longer IC1A.I0, IC1B.I0, IC2A.I0, IC2B.I0
- net -R3-LDSEL: now also IC47C.I0, IC47D.I0; no longer IC17C.I0, IC17D.I0
- net -R3-RDSEL: now also IC26C.I0, IC26D.I0, IC47A.I0, IC47B.I0; no longer IC17A.I0, IC17B.I0, IC2C.I0, IC2D.I0
- net -REG-DN: now also IC15B.I1, IC25B.I1, IC47B.I1; no longer IC17B.I1, IC24B.I1, IC9B.I1
- net -REG-LD-HI: now also IC15D.I1, IC25D.I1, IC47D.I1; no longer IC17D.I1, IC24D.I1, IC9D.I1
- net -REG-LD-LO: now also IC15C.I1, IC25C.I1, IC47C.I1; no longer IC17C.I1, IC24C.I1, IC9C.I1
- net -REG-RD-HI: now also IC26B.I1, IC26D.I1; no longer IC10B.I1, IC10D.I1
- net -REG-RD-LO: now also IC26A.I1, IC26C.I1; no longer IC10A.I1, IC10C.I1
- net -REG-UP: now also IC15A.I1, IC25A.I1, IC47A.I1; no longer IC17A.I1, IC24A.I1, IC9A.I1
- net ADATA0: now also IC13B.Y1, IC19A.A, IC23B.Y1, IC29A.A, IC45B.Y1, IC9A.A; no longer IC11A.A, IC15B.Y1, IC18A.A, IC22B.Y1, IC25A.A, IC29B.Y1
- net ADATA1: now also IC13B.Y2, IC19A.B, IC23B.Y2, IC29A.B, IC45B.Y2, IC9A.B; no longer IC11A.B, IC15B.Y2, IC18A.B, IC22B.Y2, IC25A.B, IC29B.Y2
- net ADATA10: now also IC11A.C, IC14B.Y3, IC21A.C, IC24B.Y3, IC43A.C, IC46B.Y3; no longer IC13A.C, IC16B.Y3, IC20A.C, IC23B.Y3, IC27A.C, IC30B.Y3
- net ADATA11: now also IC11A.D, IC14B.Y4, IC21A.D, IC24B.Y4, IC43A.D, IC46B.Y4; no longer IC13A.D, IC16B.Y4, IC20A.D, IC23B.Y4, IC27A.D, IC30B.Y4
- net ADATA12: now also IC12A.A, IC14A.Y1, IC22A.A, IC24A.Y1, IC44A.A, IC46A.Y1; no longer IC14A.A, IC16A.Y1, IC21A.A, IC23A.Y1, IC28A.A, IC30A.Y1
- net ADATA13: now also IC12A.B, IC14A.Y2, IC22A.B, IC24A.Y2, IC44A.B, IC46A.Y2; no longer IC14A.B, IC16A.Y2, IC21A.B, IC23A.Y2, IC28A.B, IC30A.Y2
- net ADATA14: now also IC12A.C, IC14A.Y3, IC22A.C, IC24A.Y3, IC44A.C, IC46A.Y3; no longer IC14A.C, IC16A.Y3, IC21A.C, IC23A.Y3, IC28A.C, IC30A.Y3
- net ADATA15: now also IC12A.D, IC14A.Y4, IC22A.D, IC24A.Y4, IC44A.D, IC46A.Y4; no longer IC14A.D, IC16A.Y4, IC21A.D, IC23A.Y4, IC28A.D, IC30A.Y4
- net ADATA2: now also IC13B.Y3, IC19A.C, IC23B.Y3, IC29A.C, IC45B.Y3, IC9A.C; no longer IC11A.C, IC15B.Y3, IC18A.C, IC22B.Y3, IC25A.C, IC29B.Y3
- net ADATA3: now also IC13B.Y4, IC19A.D, IC23B.Y4, IC29A.D, IC45B.Y4, IC9A.D; no longer IC11A.D, IC15B.Y4, IC18A.D, IC22B.Y4, IC25A.D, IC29B.Y4
- net ADATA4: now also IC10A.A, IC13A.Y1, IC20A.A, IC23A.Y1, IC30A.A, IC45A.Y1; no longer IC12A.A, IC15A.Y1, IC19A.A, IC22A.Y1, IC26A.A, IC29A.Y1
- net ADATA5: now also IC10A.B, IC13A.Y2, IC20A.B, IC23A.Y2, IC30A.B, IC45A.Y2; no longer IC12A.B, IC15A.Y2, IC19A.B, IC22A.Y2, IC26A.B, IC29A.Y2
- net ADATA6: now also IC10A.C, IC13A.Y3, IC20A.C, IC23A.Y3, IC30A.C, IC45A.Y3; no longer IC12A.C, IC15A.Y3, IC19A.C, IC22A.Y3, IC26A.C, IC29A.Y3
- net ADATA7: now also IC10A.D, IC13A.Y4, IC20A.D, IC23A.Y4, IC30A.D, IC45A.Y4; no longer IC12A.D, IC15A.Y4, IC19A.D, IC22A.Y4, IC26A.D, IC29A.Y4
- net ADATA8: now also IC11A.A, IC14B.Y1, IC21A.A, IC24B.Y1, IC43A.A, IC46B.Y1; no longer IC13A.A, IC16B.Y1, IC20A.A, IC23B.Y1, IC27A.A, IC30B.Y1
- net ADATA9: now also IC11A.B, IC14B.Y2, IC21A.B, IC24B.Y2, IC43A.B, IC46B.Y2; no longer IC13A.B, IC16B.Y2, IC20A.B, IC23B.Y2, IC27A.B, IC30B.Y2
- net ADDR0: now also IC17A.Y1, IC27A.Y1, IC41A.Y1, IC49A.Y1
- net ADDR1: now also IC17A.Y2, IC27A.Y2, IC41A.Y2, IC49A.Y2
- net ADDR10: now also IC18A.Y3, IC28A.Y3, IC42A.Y3, IC50A.Y3
- net ADDR11: now also IC18A.Y4, IC28A.Y4, IC42A.Y4, IC50A.Y4
- net ADDR12: now also IC18B.Y1, IC28B.Y1, IC42B.Y1, IC50B.Y1
- net ADDR13: now also IC18B.Y2, IC28B.Y2, IC42B.Y2, IC50B.Y2
- net ADDR14: now also IC18B.Y3, IC28B.Y3, IC42B.Y3, IC50B.Y3
- net ADDR15: now also IC18B.Y4, IC28B.Y4, IC42B.Y4, IC50B.Y4
- net ADDR2: now also IC17A.Y3, IC27A.Y3, IC41A.Y3, IC49A.Y3
- net ADDR3: now also IC17A.Y4, IC27A.Y4, IC41A.Y4, IC49A.Y4
- net ADDR4: now also IC17B.Y1, IC27B.Y1, IC41B.Y1, IC49B.Y1
- net ADDR5: now also IC17B.Y2, IC27B.Y2, IC41B.Y2, IC49B.Y2
- net ADDR6: now also IC17B.Y3, IC27B.Y3, IC41B.Y3, IC49B.Y3
- net ADDR7: now also IC17B.Y4, IC27B.Y4, IC41B.Y4, IC49B.Y4
- net ADDR8: now also IC18A.Y1, IC28A.Y1, IC42A.Y1, IC50A.Y1
- net ADDR9: now also IC18A.Y2, IC28A.Y2, IC42A.Y2, IC50A.Y2
- net GND: no longer JP1.1, JP1.2, JP1.39, JP1.40, JP2.1, JP2.2, JP2.39, JP2.40
- net N$115: now also IC41A.A1
- net N$116: now also IC41A.A2
- net N$117: now also IC41A.A3
- net N$118: now also IC41A.A4
- net N$119: now also IC41B.A1
- net N$120: now also IC41B.A2
- net N$121: now also IC41B.A3
- net N$122: now also IC41B.A4
- net N$123: now also IC42A.A1
- net N$124: now also IC42A.A2
- net N$125: now also IC42A.A3
- net N$126: now also IC42A.A4
- net N$127: now also IC42B.A1
- net N$128: now also IC42B.A2
- net N$129: now also IC42B.A3
- net N$130: now also IC42B.A4
- net N$2: now also IC10A.DN, IC9A.BO; no longer IC25A.BO, IC26A.DN
- net N$23: now also IC15B.O, IC9A.DN; no longer IC24B.O, IC25A.DN
- net N$25: now also IC13A.G, IC13B.G, IC2C.O; no longer IC10C.O, IC29A.G, IC29B.G
- net N$26: now also IC14A.G, IC14B.G, IC2D.O; no longer IC10D.O, IC30A.G, IC30B.G
- net N$27: now also IC11A.LD, IC12A.LD, IC15D.O; no longer IC24D.O, IC27A.LD, IC28A.LD
- net N$3: now also IC10A.UP, IC9A.CO; no longer IC25A.CO, IC26A.UP
- net N$30: now also IC13B.A3, IC17A.A3, IC9A.QC; no longer IC12A.BO, IC13A.DN
- net N$31: now also IC13B.A4, IC17A.A4, IC9A.QD; no longer IC12A.CO, IC13A.UP
- net N$32: now also IC10A.QA, IC13A.A1, IC17B.A1; no longer IC13A.BO, IC14A.DN
- net N$33: now also IC10A.QB, IC13A.A2, IC17B.A2; no longer IC13A.CO, IC14A.UP
- net N$34: now also IC10A.QC, IC13A.A3, IC17B.A3; no longer IC11A.LD, IC12A.LD, IC9C.O
- net N$35: now also IC10A.QD, IC13A.A4, IC17B.A4; no longer IC11A.UP, IC9A.O
- net N$36: now also IC11A.QA, IC14B.A1, IC18A.A1; no longer IC11A.DN, IC9B.O
- net N$38: now also IC11A.QB, IC14B.A2, IC18A.A2; no longer IC10A.O, IC15A.G, IC15B.G
- net N$39: now also IC11A.QC, IC14B.A3, IC18A.A3; no longer IC10B.O, IC16A.G, IC16B.G
- net N$4: now also IC10A.BO, IC11A.DN; no longer IC26A.BO, IC27A.DN
- net N$40: now also IC11A.QD, IC14B.A4, IC18A.A4; no longer IC13A.LD, IC14A.LD, IC9D.O
- net N$5: now also IC10A.CO, IC11A.UP; no longer IC26A.CO, IC27A.UP
- net N$64: now also IC20A.LD, IC25C.O; no longer IC17C.O, IC18A.LD
- net N$65: now also IC19A.UP, IC25A.O; no longer IC17A.O, IC18A.UP
- net N$66: now also IC19A.DN, IC25B.O; no longer IC17B.O, IC18A.DN
- net N$8: now also IC10A.LD, IC15C.O, IC9A.LD; no longer IC24C.O, IC25A.LD, IC26A.LD
- net N$80: now also IC21A.QC, IC24B.A3, IC28A.A3; no longer IC18A.QA, IC22B.A1
- net N$81: now also IC21A.QD, IC24B.A4, IC28A.A4; no longer IC18A.QB, IC22B.A2
- net N$82: now also IC22A.QA, IC24A.A1, IC28B.A1; no longer IC18A.QC, IC22B.A3
- net N$83: now also IC22A.QB, IC24A.A2, IC28B.A2; no longer IC18A.QD, IC22B.A4
- net N$84: now also IC22A.QC, IC24A.A3, IC28B.A3; no longer IC22A.G, IC22B.G, IC2C.O
- net N$85: now also IC22A.QD, IC24A.A4, IC28B.A4; no longer IC23A.G, IC23B.G, IC2D.O
- net N$86: now also IC29A.BO, IC30A.DN; no longer IC17D.O, IC20A.LD, IC21A.LD
- net N$87: now also IC29A.CO, IC30A.UP; no longer IC19A.QA, IC22A.A1
- net N$88: now also IC30A.BO, IC43A.DN; no longer IC19A.QB, IC22A.A2
- net N$89: now also IC30A.CO, IC43A.UP; no longer IC19A.QC, IC22A.A3
- net N$9: now also IC15A.O, IC9A.UP; no longer IC24A.O, IC25A.UP
- net N$90: now also IC43A.BO, IC44A.DN; no longer IC19A.QD, IC22A.A4
- net N$91: now also IC43A.CO, IC44A.UP; no longer IC20A.QA, IC23B.A1
- net N$92: now also IC29A.LD, IC30A.LD, IC47C.O; no longer IC20A.QB, IC23B.A2
- net N$93: now also IC29A.UP, IC47A.O; no longer IC20A.QC, IC23B.A3
- net N$94: now also IC29A.DN, IC47B.O; no longer IC20A.QD, IC23B.A4
- net N$95: now also IC26C.O, IC45A.G, IC45B.G; no longer IC21A.QA, IC23A.A1
- net N$96: now also IC26D.O, IC46A.G, IC46B.G; no longer IC21A.QB, IC23A.A2
- net N$97: now also IC43A.LD, IC44A.LD, IC47D.O; no longer IC21A.QC, IC23A.A3
- net N$98: now also IC29A.QA, IC45B.A1, IC49A.A1; no longer IC21A.QD, IC23A.A4
- net RESET: now also IC10A.CLR, IC22A.CLR, IC29A.CLR, IC30A.CLR, IC43A.CLR, IC44A.CLR, IC9A.CLR; no longer IC13A.CLR, IC14A.CLR, IC18A.CLR, IC25A.CLR, IC26A.CLR, IC27A.CLR, IC28A.CLR
