File: PCB/Working - Under Develolpment/Memory v1.2/Memory V1.2.brd (EAGLE design)
At the start: 177.8 x 114 mm, 19 parts, among them IC10 74ALS00N, IC11 74LS157N, IC12 74LS74N, IC4 74ALS30N, IC5 74LS245N, IC6 74LS04N, IC7 74LS138N, IC8 74LS244N, IC9 74LS244N, X1 FABC96R

Commit message: Ongoing development
Parts:
- added C1, C10, C11, C12, C13, C14, C15, C16, C17, C18, C2, C3, C4, C5, C6, C7, C8, C9: (no value), adafruit:C025-025X050
- added IC13: (no value), memory-nec:DIL28-6
- added IC14: 74LS04N, 74xx-us:DIL14
- added IC15, IC16, IC17, IC19: 74LS374N, 74xx-us:DIL20
- added JP1: (no value), pinhead:1X03
- added RN5, RN6: (no value), resistor-net:RN-9
- IC3: value (none) -> 74LS32N; device memory:DIL24 -> 74xx-us:DIL14
- moved IC3 79.0 mm to (33.0, 21.6)
- moved RN1 7.62 mm to (108.0, 16.5)
- moved RN2 1.27 mm to (108.0, 47.0)
Connections:
- net -ADDR-REG-LD0 renamed -ADDR-REG-ID1
- net -ADDR-REG-LD1 renamed -ADDR-REG-ID3
- net -ADDR-REG-RD0 renamed -ADDR-REG-ID0
- net -ADDR-REG-RD1 renamed -ADDR-REG-ID2
- removed net -ROM: IC3.18, IC7.7
- new net -ROM-CS: IC13.20, IC6.12
- new net -ROME000: IC10.12, IC7.9
- new net -ROMF000: IC10.13, IC7.7
- new net N$19: IC10.8, IC12.3
- new net N$20: IC10.10, IC10.6, IC10.9
- new net N$21: IC14.6, IC15.11, IC16.11
- new net N$22: IC10.5, IC14.2
- new net N$23: IC14.8, IC17.11, IC19.11
- new net N$24: IC7.5, JP1.2
- new net N$25: IC14.1, IC3.3
- net -BUS-EN: now also IC3.2, JP1.1
- net -TMP-REG-LD0: now also IC14.5
- net -TMP-REG-LD1: now also IC14.9
- net -TMP-REG-RD0: now also IC15.1, IC16.1
- net -TMP-REG-RD1: now also IC17.1, IC19.1
- net -VMA: now also IC14.11, IC3.1; no longer IC10.10, IC10.9
- net ADDR15: now also IC10.4; no longer IC12.3
- net BADDR0: now also IC13.10; no longer IC3.8
- net BADDR1: now also IC13.9; no longer IC3.7
- net BADDR10: now also IC13.21; no longer IC3.19
- net BADDR11: now also IC13.23; no longer IC3.21
- net BADDR12: now also IC13.2
- net BADDR15: now also IC14.3; no longer IC10.4, IC10.5
- net BADDR2: now also IC13.8; no longer IC3.6
- net BADDR3: now also IC13.7; no longer IC3.5
- net BADDR4: now also IC13.6; no longer IC3.4
- net BADDR5: now also IC13.5; no longer IC3.3
- net BADDR6: now also IC13.4; no longer IC3.2
- net BADDR7: now also IC13.3; no longer IC3.1
- net BADDR8: now also IC13.25; no longer IC3.23
- net BADDR9: now also IC13.24; no longer IC3.22
- net BDATA0: now also IC13.11; no longer IC3.9
- net BDATA1: now also IC13.12; no longer IC3.10
- net BDATA2: now also IC13.13; no longer IC3.11
- net BDATA3: now also IC13.15; no longer IC3.13
- net BDATA4: now also IC13.16; no longer IC3.14
- net BDATA5: now also IC13.17; no longer IC3.15
- net BDATA6: now also IC13.18; no longer IC3.16
- net BDATA7: now also IC13.19; no longer IC3.17
- net DATA0: now also IC15.2, IC15.3, IC17.2, IC17.3, RN5.2
- net DATA1: now also IC15.4, IC15.5, IC17.4, IC17.5, RN5.3
- net DATA10: now also IC16.6, IC16.7, IC19.6, IC19.7, RN6.4
- net DATA11: now also IC16.8, IC16.9, IC19.8, IC19.9, RN6.5
- net DATA12: now also IC16.12, IC16.13, IC19.12, IC19.13, RN6.6
- net DATA13: now also IC16.14, IC16.15, IC19.14, IC19.15, RN6.7
- net DATA14: now also IC16.16, IC16.17, IC19.16, IC19.17, RN6.8
- net DATA15: now also IC16.18, IC16.19, IC19.18, IC19.19, RN6.9
- net DATA2: now also IC15.6, IC15.7, IC17.6, IC17.7, RN5.4
- net DATA3: now also IC15.8, IC15.9, IC17.8, IC17.9, RN5.5
- net DATA4: now also IC15.12, IC15.13, IC17.12, IC17.13, RN5.6
- net DATA5: now also IC15.14, IC15.15, IC17.14, IC17.15, RN5.7
- net DATA6: now also IC15.16, IC15.17, IC17.16, IC17.17, RN5.8
- net DATA7: now also IC15.18, IC15.19, IC17.18, IC17.19, RN5.9
- net DATA8: now also IC16.2, IC16.3, IC19.2, IC19.3, RN6.2
- net DATA9: now also IC16.4, IC16.5, IC19.4, IC19.5, RN6.3
- net GND: now also C1.2, C10.2, C11.2, C12.2, C13.2, C14.2, C15.2, C16.2, C17.2, C18.2, C2.2, C3.2, C4.2, C5.2, C6.2, C7.2, C8.2, C9.2, IC13.14, IC14.13, IC14.7, IC15.10, IC16.10, IC17.10, IC19.10, IC3.10, IC3.13, IC3.4, IC3.5, IC3.7, IC3.9, JP1.3, RN5.1, RN6.1; no longer IC10.12, IC10.13, IC6.13, IC7.5
- net N$1: now also IC10.11, IC6.13; no longer IC4.12, IC7.9
- net N$12: now also IC14.10; no longer IC10.8
- net N$13: now also IC14.4; no longer IC10.6
- net N$3: now also IC13.22; no longer IC3.20
- net N$4: now also IC13.27
- net VCC: now also C1.1, C10.1, C11.1, C12.1, C13.1, C14.1, C15.1, C16.1, C17.1, C18.1, C2.1, C3.1, C4.1, C5.1, C6.1, C7.1, C8.1, C9.1, IC13.28, IC14.14, IC15.20, IC16.20, IC17.20, IC19.20, IC3.14, IC4.12; no longer IC3.24
Routing:
- net GND: track 565.9 -> 0.00 mm
- net VCC: track 494.0 -> 0.00 mm
- net DATA9: track 0.00 -> 289.7 mm, vias 0 -> 1
- net DATA11: track 0.00 -> 274.5 mm
- net DATA10: track 0.00 -> 262.3 mm
- net DATA12: track 0.00 -> 238.8 mm
- net DATA14: track 0.00 -> 238.5 mm, vias 0 -> 1
- net DATA13: track 0.00 -> 237.3 mm
- net DATA8: track 0.00 -> 217.5 mm, vias 0 -> 2
- net DATA15: track 0.00 -> 203.5 mm, vias 0 -> 2
- net N$21: track 0.00 -> 191.0 mm, vias 0 -> 1
- net -TMP-REG-RD0: track 0.00 -> 185.9 mm
- net -TMP-REG-RD1: track 0.00 -> 176.0 mm, vias 0 -> 1
- net DATA4: track 94.0 -> 263.4 mm
- net DATA0: track 63.2 -> 227.3 mm
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- added copper zone on layer 2, net GND
- added copper zone on layer 15, net VCC
Other:
- board text added: "-BUS-EN"
- board text added: "Gnd"
