File: PCB/Working - Under Develolpment/Memory v1.2/Memory V1.2.sch (EAGLE design)
At the start: 19 parts, among them IC10 74ALS00N, IC11 74LS157N, IC12 74LS74N, IC4 74ALS30N, IC5 74LS245N, IC6 74LS04N, IC7 74LS138N, IC8 74LS244N, IC9 74LS244N, X1 FABC96R

Commit message: Ongoing development
Parts:
- added C1, C10, C11, C12, C13, C14, C15, C16, C17, C18, C2, C3, C4, C5, C6, C7, C8, C9: (no value), adafruit:C-US025-025X050
- added IC13: (no value), memory-nec:28C64C
- added IC14: 74LS04N, 74xx-us:74LS04N
- added IC15, IC16, IC17, IC19: 74LS374N, 74xx-us:74LS374N
- added JP1: (no value), pinhead:PINHD-1X3
- added RN5, RN6: (no value), resistor-net:RNX8
- IC3: value (none) -> 74LS32N; device memory:2732 -> 74xx-us:74LS32N
Connections:
- net -ADDR-REG-LD0 renamed -ADDR-REG-ID1
- net -ADDR-REG-LD1 renamed -ADDR-REG-ID3
- net -ADDR-REG-RD0 renamed -ADDR-REG-ID0
- net -ADDR-REG-RD1 renamed -ADDR-REG-ID2
- removed net -ROM: IC3A.!CE, IC7A.Y7
- new net -ROM-CS: IC13.!CE, IC6F.O
- new net -ROME000: IC10D.I0, IC7A.Y6
- new net -ROMF000: IC10D.I1, IC7A.Y7
- new net N$19: IC10C.O, IC12A.CLK
- new net N$20: IC10B.O, IC10C.I0, IC10C.I1
- new net N$21: IC14C.O, IC15A.CLK, IC16A.CLK
- new net N$22: IC10B.I1, IC14A.O
- new net N$23: IC14D.O, IC17A.CLK, IC19A.CLK
- new net N$24: IC7A.G2B, JP1.2
- new net N$25: IC14A.I, IC3A.O
- net -BUS-EN: now also IC3A.I1, JP1.1
- net -TMP-REG-LD0: now also IC14C.I
- net -TMP-REG-LD1: now also IC14D.I
- net -TMP-REG-RD0: now also IC15A.OC, IC16A.OC
- net -TMP-REG-RD1: now also IC17A.OC, IC19A.OC
- net -VMA: now also IC14E.I, IC3A.I0; no longer IC10C.I0, IC10C.I1
- net ADDR15: now also IC10B.I0; no longer IC12A.CLK
- net BADDR0: now also IC13.A0; no longer IC3A.A0
- net BADDR1: now also IC13.A1; no longer IC3A.A1
- net BADDR10: now also IC13.A10; no longer IC3A.A10
- net BADDR11: now also IC13.A11; no longer IC3A.A11
- net BADDR12: now also IC13.A12
- net BADDR15: now also IC14B.I; no longer IC10B.I0, IC10B.I1
- net BADDR2: now also IC13.A2; no longer IC3A.A2
- net BADDR3: now also IC13.A3; no longer IC3A.A3
- net BADDR4: now also IC13.A4; no longer IC3A.A4
- net BADDR5: now also IC13.A5; no longer IC3A.A5
- net BADDR6: now also IC13.A6; no longer IC3A.A6
- net BADDR7: now also IC13.A7; no longer IC3A.A7
- net BADDR8: now also IC13.A8; no longer IC3A.A8
- net BADDR9: now also IC13.A9; no longer IC3A.A9
- net BDATA0: now also IC13.I/O0; no longer IC3A.O0
- net BDATA1: now also IC13.I/O1; no longer IC3A.O1
- net BDATA2: now also IC13.I/O2; no longer IC3A.O2
- net BDATA3: now also IC13.I/O3; no longer IC3A.O3
- net BDATA4: now also IC13.I/O4; no longer IC3A.O4
- net BDATA5: now also IC13.I/O5; no longer IC3A.O5
- net BDATA6: now also IC13.I/O6; no longer IC3A.O6
- net BDATA7: now also IC13.I/O7; no longer IC3A.O7
- net DATA0: now also IC15A.1D, IC15A.1Q, IC17A.1D, IC17A.1Q, RN5-1.1
- net DATA1: now also IC15A.2D, IC15A.2Q, IC17A.2D, IC17A.2Q, RN5-2.1
- net DATA10: now also IC16A.3D, IC16A.3Q, IC19A.3D, IC19A.3Q, RN6-3.1
- net DATA11: now also IC16A.4D, IC16A.4Q, IC19A.4D, IC19A.4Q, RN6-4.1
- net DATA12: now also IC16A.5D, IC16A.5Q, IC19A.5D, IC19A.5Q, RN6-5.1
- net DATA13: now also IC16A.6D, IC16A.6Q, IC19A.6D, IC19A.6Q, RN6-6.1
- net DATA14: now also IC16A.7D, IC16A.7Q, IC19A.7D, IC19A.7Q, RN6-7.1
- net DATA15: now also IC16A.8D, IC16A.8Q, IC19A.8D, IC19A.8Q, RN6-8.1
- net DATA2: now also IC15A.3D, IC15A.3Q, IC17A.3D, IC17A.3Q, RN5-3.1
- net DATA3: now also IC15A.4D, IC15A.4Q, IC17A.4D, IC17A.4Q, RN5-4.1
- net DATA4: now also IC15A.5D, IC15A.5Q, IC17A.5D, IC17A.5Q, RN5-5.1
- net DATA5: now also IC15A.6D, IC15A.6Q, IC17A.6D, IC17A.6Q, RN5-6.1
- net DATA6: now also IC15A.7D, IC15A.7Q, IC17A.7D, IC17A.7Q, RN5-7.1
- net DATA7: now also IC15A.8D, IC15A.8Q, IC17A.8D, IC17A.8Q, RN5-8.1
- net DATA8: now also IC16A.1D, IC16A.1Q, IC19A.1D, IC19A.1Q, RN6-1.1
- net DATA9: now also IC16A.2D, IC16A.2Q, IC19A.2D, IC19A.2Q, RN6-2.1
- net GND: now also C1.2, C10.2, C11.2, C12.2, C13.2, C14.2, C15.2, C16.2, C17.2, C18.2, C2.2, C3.2, C4.2, C5.2, C6.2, C7.2, C8.2, C9.2, IC13.GND, IC14F.I, IC3B.I0, IC3B.I1, IC3C.I0, IC3C.I1, IC3D.I0, IC3D.I1, JP1.3, RN5_.1, RN6_.1; no longer IC10D.I0, IC10D.I1, IC6F.I, IC7A.G2B
- net N$1: now also IC10D.O, IC6F.I; no longer IC4A.I7, IC7A.Y6
- net N$12: now also IC14E.O; no longer IC10C.O
- net N$13: now also IC14B.O; no longer IC10B.O
- net N$3: now also IC13.!OE; no longer IC3A.!OE!/VPP
- net N$4: now also IC13.!WE
- net VCC: now also C1.1, C10.1, C11.1, C12.1, C13.1, C14.1, C15.1, C16.1, C17.1, C18.1, C2.1, C3.1, C4.1, C5.1, C6.1, C7.1, C8.1, C9.1, IC13.VCC, IC4A.I7
