File: PCB/Working - Under Develolpment/Address and TMP-V1.0/Address and TMP V1.0.sch (EAGLE design)
At the start: 16 parts, among them IC1 74LS373N, IC2 74LS373N, IC3 74LS373N, IC4 74LS373N, IC5 74LS04N, IC6 74LS373N, IC7 74LS373N, IC8 74LS373N, IC9 74LS373N, X1 FABC96R

Commit message: testing gitignore
Other:
- note added: "test text"
Changed lines of the file:
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@@
 <description>BUS</description>
 <plain>
+<text x="10.16" y="99.06" size="1.778" layer="91">test text</text>
 </plain>
 <instances>
