File: PCB/Working - Under Develolpment/ALU-V3.3/ALU V3.2.sch (EAGLE design)
At the start: 84 parts, among them IC1 74ALS04N, IC10 74LS245N, IC11 74LS245N, IC12 74LS244N, IC13 74LS244N, IC14 74LS86N, IC15 74LS86N, IC16 74LS244N, IC17 74LS244N, IC18 74LS08N, IC19 74LS08N, IC2 74LS240N, IC20 74LS244N, IC21 74LS32N, IC22 74LS32N, IC23 74LS244N, IC24 74LS85N, IC25 74LS85N, IC26 74LS251N, IC27 74LS86N, IC28 74LS153N, IC29 74LS194N, IC3 74LS244N, IC30 74LS194N, IC31 74LS244N, IC32 74LS153N, IC33 74LS86N, IC34 74LS86N, IC35 74LS283N, IC36 74LS283N, IC37 74LS244N, IC4 74LS00N, IC5 74LS374N, IC6 74ALS08N, IC7 74LS32N, IC8 74LS138N, IC9 74LS74N, X1 FABC96R

Commit message: Next version of ALU to production
Parts:
- added JP1, JP2: (no value), pinhead:PINHD-1X3
Connections:
- net UNUSED0 renamed -VMA
- removed net -BUS-OUT: IC10A.DIR, IC11A.DIR, IC1D.O
- removed net N$57: IC29A.QA, IC31A.A1, IC32A.1C1
- removed net N$74: IC30A.QD, IC31B.A4, IC32A.1C2
- new net N$10: IC27B.O, IC4B.I1
- new net N$15: IC1D.O, IC4B.I0
- new net N$16: IC1E.I, IC4B.O
- new net N$4: IC26A.G, JP1.2
- new net N$9: IC6C.I1, JP2.2
- new net SRD0: IC28A.2C1, IC29A.QA, IC31A.A1, IC32A.1C2
- new net SRD7: IC28A.1C1, IC30A.QD, IC31B.A4, IC32A.1C1
- net -AC-LD: now also JP2.1; no longer IC1D.I
- net -AC-RD: now also IC10A.DIR, IC11A.DIR
- net -ADD/SUB: now also IC1D.I
- net -ALU-FUNC: now also JP1.1
- net AC-LD: now also JP2.3; no longer IC6C.I1
- net ACO-DATA0: now also IC35A.A1; no longer IC28A.2C1, IC33A.I0
- net ACO-DATA1: now also IC35A.A2; no longer IC33B.I0
- net ACO-DATA2: now also IC35A.A3; no longer IC33C.I0
- net ACO-DATA3: now also IC35A.A4; no longer IC33D.I0
- net ACO-DATA4: now also IC36A.A1; no longer IC34A.I0
- net ACO-DATA5: now also IC36A.A2; no longer IC34B.I0
- net ACO-DATA6: now also IC36A.A3; no longer IC34C.I0
- net ACO-DATA7: now also IC36A.A4; no longer IC28A.1C1, IC34D.I0
- net BDATA0: now also IC33A.I0; no longer IC35A.A1
- net BDATA1: now also IC33B.I0; no longer IC35A.A2
- net BDATA2: now also IC33C.I0; no longer IC35A.A3
- net BDATA3: now also IC33D.I0; no longer IC35A.A4
- net BDATA4: now also IC34A.I0; no longer IC36A.A1
- net BDATA5: now also IC34B.I0; no longer IC36A.A2
- net BDATA6: now also IC34C.I0; no longer IC36A.A3
- net BDATA7: now also IC34D.I0; no longer IC36A.A4
- net CO/BO: now also IC1E.O; no longer IC27B.O
- net GND: now also JP1.3; no longer IC1E.I, IC26A.G, IC4B.I0, IC4B.I1
Other:
- moved on the sheet: IC27B, IC6D
