File: PCB/Production/ALU-V3.2/ALU V3.2.brd (EAGLE design)
At the start: 177.8 x 114 mm, 86 parts, among them IC1 74ALS04N, IC10 74LS245N, IC11 74LS245N, IC12 74LS244N, IC13 74LS244N, IC14 74LS86N, IC15 74LS86N, IC16 74LS244N, IC17 74LS244N, IC18 74LS08N, IC19 74LS08N, IC2 74LS240N, IC20 74LS244N, IC21 74LS32N, IC22 74LS32N, IC23 74LS244N, IC24 74LS85N, IC25 74LS85N, IC26 74LS251N, IC27 74LS86N, IC28 74LS153N, IC29 74LS194N, IC3 74LS244N, IC30 74LS194N, IC31 74LS244N, IC32 74LS153N, IC33 74LS86N, IC34 74LS86N, IC35 74LS283N, IC36 74LS283N, IC37 74LS244N, IC4 74LS00N, IC5 74LS374N, IC6 74ALS08N, IC7 74LS32N, IC8 74LS138N, IC9 74LS74N, X1 FABC96R

Commit message: Rename Connector C3-C6, ADDR-REG-ID0-3
Rename Connector C3-C6, ADDR-REG-ID0-3
Connections:
- net -ADDR-REG-LD0 renamed ADDR-REG-ID1
- net -ADDR-REG-LD1 renamed ADDR-REG-ID3
- net -ADDR-REG-RD0 renamed ADDR-REG-ID0
- net -ADDR-REG-RD1 renamed ADDR-REG-ID2
Changed lines of the file:
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@@
 <contactref element="X1" pad="B29"/>
 </signal>
-<signal name="-ADDR-REG-RD0">
+<signal name="ADDR-REG-ID0">
 <contactref element="X1" pad="C3"/>
 </signal>
-<signal name="-ADDR-REG-LD0">
+<signal name="ADDR-REG-ID1">
 <contactref element="X1" pad="C4"/>
 </signal>
-<signal name="-ADDR-REG-RD1">
+<signal name="ADDR-REG-ID2">
 <contactref element="X1" pad="C5"/>
 </signal>
-<signal name="-ADDR-REG-LD1">
+<signal name="ADDR-REG-ID3">
 <contactref element="X1" pad="C6"/>
 </signal>
