File: PCB/Production/Memory v1.2/Memory V1.2.brd (EAGLE design)
At the start: 177.8 x 114 mm, 46 parts, among them IC10 74ALS00N, IC11 74LS157N, IC12 74LS74N, IC14 74LS04N, IC15 74LS374N, IC16 74LS374N, IC17 74LS374N, IC19 74LS374N, IC3 74LS32N, IC4 74ALS30N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

Commit message: cleanup bus names
Connections:
- net -ADDR-REG-ID0 renamed ADDR-REG-ID0
- net -ADDR-REG-ID1 renamed ADDR-REG-ID1
- net -ADDR-REG-ID2 renamed ADDR-REG-ID2
- net -ADDR-REG-ID3 renamed ADDR-REG-ID3
- net -IN renamed IN
- net -OUT renamed OUT
Changed lines of the file:
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@@
 <via x="14.605" y="87.63" extent="1-16" drill="0.254"/>
 </signal>
-<signal name="-ADDR-REG-ID0">
+<signal name="ADDR-REG-ID0">
 <contactref element="X1" pad="C3"/>
 </signal>
-<signal name="-ADDR-REG-ID1">
+<signal name="ADDR-REG-ID1">
 <contactref element="X1" pad="C4"/>
 </signal>
-<signal name="-ADDR-REG-ID2">
+<signal name="ADDR-REG-ID2">
 <contactref element="X1" pad="C5"/>
 </signal>
-<signal name="-ADDR-REG-ID3">
+<signal name="ADDR-REG-ID3">
 <contactref element="X1" pad="C6"/>
 </signal>
@@
 <wire x1="10.16" y1="86.36" x2="11.43" y2="86.36" width="0.1524" layer="1"/>
 </signal>
-<signal name="-OUT">
+<signal name="OUT">
 <contactref element="X1" pad="C27"/>
 </signal>
-<signal name="-IN">
+<signal name="IN">
 <contactref element="X1" pad="C26"/>
 </signal>
