File: PCB/Production/Memory v1.2/Memory V1.2.sch (EAGLE design)
At the start: 46 parts, among them IC10 74ALS00N, IC11 74LS157N, IC12 74LS74N, IC14 74LS04N, IC15 74LS374N, IC16 74LS374N, IC17 74LS374N, IC19 74LS374N, IC3 74LS32N, IC4 74ALS30N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

Commit message: cleanup bus names
Connections:
- net -ADDR-REG-ID0 renamed ADDR-REG-ID0
- net -ADDR-REG-ID1 renamed ADDR-REG-ID1
- net -ADDR-REG-ID2 renamed ADDR-REG-ID2
- net -ADDR-REG-ID3 renamed ADDR-REG-ID3
- net -IN renamed IN
- net -OUT renamed OUT
Changed lines of the file:
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@@
 </instances>
 <busses>
-<bus name="MAINBUS:-AC-LD,-AC-LD-INV,-AC-RD,ADDR[0..15],-ADDR-REG-LD[0..1],-ADDR-REG-RD[0..1],ALU[0..3],-ALU-FUNC,BR-COND,-BUS-EN,DATA[0..15],-HL-SWAP,-IN,-INT,-INTA,IO-ADDR[0..3],-IO-ADDR-LD,-IO-RD,-IO-WR,-MEM-RD,-MEM-WR,-OUT,-REG-DN,-REG-FUNC-LD,-REG-FUNC-RD,-REG-LD-HI,REG-LD-ID[0..3],-REG-LD-LO,-REG-RD-HI,REG-RD-ID[0..3],-REG-RD-LO,-REG-UP,-RESET,-RUN,-SR-LD,-TMP-REG-LD[0..1],-TMP-REG-RD[0..1],-VMA">
+<bus name="MAINBUS:-AC-LD,-AC-LD-INV,-AC-RD,ADDR[0..15],ADDR-REG-ID0,ADDR-REG-ID1,ADDR-REG-ID2,ADDR-REG-ID3,ALU[0..3],-ALU-FUNC,BR-COND,-BUS-EN,DATA[0..15],-HL-SWAP,IN,-INT,-INTA,IO-ADDR[0..3],-IO-ADDR-LD,-IO-RD,-IO-WR,-MEM-RD,-MEM-WR,OUT,-REG-DN,-REG-FUNC-LD,-REG-FUNC-RD,-REG-LD-HI,REG-LD-ID[0..3],-REG-LD-LO,-REG-RD-HI,REG-RD-ID[0..3],-REG-RD-LO,-REG-UP,-RESET,-RUN,-SR-LD,-TMP-REG-LD[0..1],-TMP-REG-RD[0..1],-VMA">
 <segment>
 <wire x1="-33.02" y1="-1.27" x2="182.88" y2="-1.27" width="0.762" layer="92"/>
@@
 </segment>
 </net>
-<net name="-ADDR-REG-ID0" class="0">
+<net name="ADDR-REG-ID0" class="0">
 <segment>
 <pinref part="X1" gate="-C3" pin="B"/>
@@
 </segment>
 </net>
-<net name="-ADDR-REG-ID1" class="0">
+<net name="ADDR-REG-ID1" class="0">
 <segment>
 <pinref part="X1" gate="-C4" pin="B"/>
@@
 </segment>
 </net>
-<net name="-ADDR-REG-ID2" class="0">
+<net name="ADDR-REG-ID2" class="0">
 <segment>
 <pinref part="X1" gate="-C5" pin="B"/>
@@
 </segment>
 </net>
-<net name="-ADDR-REG-ID3" class="0">
+<net name="ADDR-REG-ID3" class="0">
 <segment>
 <pinref part="X1" gate="-C6" pin="B"/>
@@
 </segment>
 </net>
-<net name="-OUT" class="0">
+<net name="OUT" class="0">
 <segment>
 <pinref part="X1" gate="-C27" pin="B"/>
@@
 </segment>
 </net>
-<net name="-IN" class="0">
+<net name="IN" class="0">
 <segment>
 <pinref part="X1" gate="-C26" pin="B"/>
