File: PCB/Production/IO-V-1.1/IO V1.1.brd (EAGLE design)
At the start: 177.8 x 114 mm, 71 parts, among them IC10 74273N, IC11 74LS10N, IC2 MAX232, IC3 74LS244N, IC4 74273N, IC5 74LS138N, IC6 74LS10N, IC7 74LS00N, IC8 74LS06N, IC9 74273N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

Commit message: Cleanup Bus signals
Connections:
- net -ADDR-REG-LD0 renamed ADDR-REG-ID1
- net -ADDR-REG-LD1 renamed ADDR-REG-ID3
- net -ADDR-REG-RD0 renamed ADDR-REG-ID0
- net -ADDR-REG-RD1 renamed ADDR-REG-ID2
Changed lines of the file:
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@@
 <contactref element="X1" pad="B29"/>
 </signal>
-<signal name="-ADDR-REG-RD0">
+<signal name="ADDR-REG-ID0">
 <contactref element="X1" pad="C3"/>
 </signal>
-<signal name="-ADDR-REG-LD0">
+<signal name="ADDR-REG-ID1">
 <contactref element="X1" pad="C4"/>
 </signal>
-<signal name="-ADDR-REG-RD1">
+<signal name="ADDR-REG-ID2">
 <contactref element="X1" pad="C5"/>
 </signal>
-<signal name="-ADDR-REG-LD1">
+<signal name="ADDR-REG-ID3">
 <contactref element="X1" pad="C6"/>
 </signal>
