File: PCB/Working - Under Develolpment/Memory v1.3/Memory V1.3.brd (EAGLE design)
At the start: 177.8 x 114 mm, 55 parts, among them IC10 74ALS00N, IC11 74LS157N, IC12 74LS74N, IC14 74LS04N, IC15 74LS374N, IC16 74LS374N, IC17 74LS374N, IC18 74ALS30N, IC19 74LS374N, IC21 74LS374N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

Commit message: cleaning up paths
Parts:
- removed IC15, IC16, IC17, IC19, IC21, IC22, IC23, IC24: 74LS374N, 74xx-us:DIL20
- removed IC25: 74LS139N, 74xx-us:DIL16
- added IC26, IC27, IC28, IC29: 74LS374N, 74xx-us:DIL20
- added RN5, RN6: (no value), resistor-net:RN-9
Connections:
- removed net -TMP-REG-RD: IC25.1
- removed net -TMP-REG-WR: IC25.15
- removed net -TREG-LD0: IC25.12
- removed net -TREG-LD1: IC14.9, IC25.11
- removed net -TREG-LD2: IC14.13, IC25.10
- removed net -TREG-LD3: IC14.1, IC25.9
- removed net -TREG-LDO: IC14.5
- removed net -TREG-RD0: IC15.1, IC16.1, IC25.4
- removed net -TREG-RD1: IC17.1, IC19.1, IC25.5
- removed net -TREG-RD2: IC21.1, IC22.1, IC25.6
- removed net -TREG-RD3: IC23.1, IC24.1, IC25.7
- removed net N$21: IC14.6, IC15.11, IC16.11
- removed net N$23: IC14.8, IC17.11, IC19.11
- removed net N$45: IC14.12, IC21.11, IC22.11
- removed net N$46: IC14.2, IC23.11, IC24.11
- removed net TMP-ID0: IC25.14, IC25.2
- removed net TMP-ID1: IC25.13, IC25.3
- new net N$33: IC14.2, IC26.11, IC27.11
- new net N$47: IC14.12, IC28.11, IC29.11
- net -TMP-REG-LD0: now also IC14.1
- net -TMP-REG-LD1: now also IC14.13
- net -TMP-REG-RD0: now also IC26.1, IC27.1
- net -TMP-REG-RD1: now also IC28.1, IC29.1
- net DATA0: now also IC26.2, IC26.3, IC28.2, IC28.3, RN5.2; no longer IC15.2, IC15.3, IC17.2, IC17.3, IC21.2, IC21.3, IC23.2, IC23.3
- net DATA1: now also IC26.4, IC26.5, IC28.4, IC28.5, RN5.3; no longer IC15.4, IC15.5, IC17.4, IC17.5, IC21.4, IC21.5, IC23.4, IC23.5
- net DATA10: now also IC27.6, IC27.7, IC29.6, IC29.7, RN6.4; no longer IC16.6, IC16.7, IC19.6, IC19.7, IC22.6, IC22.7, IC24.6, IC24.7
- net DATA11: now also IC27.8, IC27.9, IC29.8, IC29.9, RN6.5; no longer IC16.8, IC16.9, IC19.8, IC19.9, IC22.8, IC22.9, IC24.8, IC24.9
- net DATA12: now also IC27.12, IC27.13, IC29.12, IC29.13, RN6.6; no longer IC16.12, IC16.13, IC19.12, IC19.13, IC22.12, IC22.13, IC24.12, IC24.13
- net DATA13: now also IC27.14, IC27.15, IC29.14, IC29.15, RN6.7; no longer IC16.14, IC16.15, IC19.14, IC19.15, IC22.14, IC22.15, IC24.14, IC24.15
- net DATA14: now also IC27.16, IC27.17, IC29.16, IC29.17, RN6.8; no longer IC16.16, IC16.17, IC19.16, IC19.17, IC22.16, IC22.17, IC24.16, IC24.17
- net DATA15: now also IC27.18, IC27.19, IC29.18, IC29.19, RN6.9; no longer IC16.18, IC16.19, IC19.18, IC19.19, IC22.18, IC22.19, IC24.18, IC24.19
- net DATA2: now also IC26.6, IC26.7, IC28.6, IC28.7, RN5.4; no longer IC15.6, IC15.7, IC17.6, IC17.7, IC21.6, IC21.7, IC23.6, IC23.7
- net DATA3: now also IC26.8, IC26.9, IC28.8, IC28.9, RN5.5; no longer IC15.8, IC15.9, IC17.8, IC17.9, IC21.8, IC21.9, IC23.8, IC23.9
- net DATA4: now also IC26.12, IC26.13, IC28.12, IC28.13, RN5.6; no longer IC15.12, IC15.13, IC17.12, IC17.13, IC21.12, IC21.13, IC23.12, IC23.13
- net DATA5: now also IC26.14, IC26.15, IC28.14, IC28.15, RN5.7; no longer IC15.14, IC15.15, IC17.14, IC17.15, IC21.14, IC21.15, IC23.14, IC23.15
- net DATA6: now also IC26.16, IC26.17, IC28.16, IC28.17, RN5.8; no longer IC15.16, IC15.17, IC17.16, IC17.17, IC21.16, IC21.17, IC23.16, IC23.17
- net DATA7: now also IC26.18, IC26.19, IC28.18, IC28.19, RN5.9; no longer IC15.18, IC15.19, IC17.18, IC17.19, IC21.18, IC21.19, IC23.18, IC23.19
- net DATA8: now also IC27.2, IC27.3, IC29.2, IC29.3, RN6.2; no longer IC16.2, IC16.3, IC19.2, IC19.3, IC22.2, IC22.3, IC24.2, IC24.3
- net DATA9: now also IC27.4, IC27.5, IC29.4, IC29.5, RN6.3; no longer IC16.4, IC16.5, IC19.4, IC19.5, IC22.4, IC22.5, IC24.4, IC24.5
- net GND: now also IC26.10, IC27.10, IC28.10, IC29.10, RN5.1, RN6.1; no longer IC15.10, IC16.10, IC17.10, IC19.10, IC21.10, IC22.10, IC23.10, IC24.10, IC25.8
- net VCC: now also IC26.20, IC27.20, IC28.20, IC29.20; no longer IC15.20, IC16.20, IC17.20, IC19.20, IC21.20, IC22.20, IC23.20, IC24.20, IC25.16
Routing:
- net N$23: track 191.0 -> 0.00 mm, vias 1 -> 0
- net N$21: track 182.6 -> 0.00 mm, vias 1 -> 0
- net N$45: track 158.3 -> 0.00 mm, vias 1 -> 0
- net N$46: track 156.7 -> 0.00 mm, vias 2 -> 0
- net -TREG-LD2: track 145.5 -> 0.00 mm
- net -TREG-RD0: track 142.6 -> 0.00 mm
- net -TREG-LD3: track 126.8 -> 0.00 mm, vias 1 -> 0
- net DATA3: track 298.3 -> 174.0 mm
- net -TREG-LD1: track 110.9 -> 0.00 mm
- net -TREG-RD1: track 101.2 -> 0.00 mm, vias 1 -> 0
- net DATA6: track 255.7 -> 156.7 mm
- net DATA7: track 254.8 -> 156.6 mm
- net DATA1: track 261.5 -> 165.6 mm
- net DATA2: track 268.3 -> 172.4 mm
- net DATA5: track 255.1 -> 160.6 mm
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