File: PCB/Working - Under Develolpment/Memory v1.3/Memory V1.3.sch (EAGLE design)
At the start: 33 parts, among them IC10 74ALS00N, IC11 74LS157N, IC12 74LS74N, IC3 74ALS00N, IC4 74ALS30N, IC5 74LS245N, IC6 74LS04N, IC7 74LS138N, IC8 74LS244N, IC9 74LS244N, X1 FABC96R

Commit message: Cleanup memory card files
Parts:
- removed RN1, RN2, RN3, RN4: (no value), resistor-net:RNX8
- added C14, C15, C16, C17, C18, C19, C20, C21, C22, C23, C24: (no value), adafruit:C-US025-025X050
- added IC14: 74LS04N, 74xx-us:74LS04N
- added IC15, IC16, IC17, IC19, IC21, IC22, IC23, IC24: 74LS374N, 74xx-us:74LS374N
- added IC18: 74ALS30N, 74xx-us:74ALS30N
- added IC25: 74LS139N, 74xx-us:74LS139N
- added JP1: (no value), pinhead:PINHD-1X3
- added RN7, RN8: (no value), resistor-sil:G08R
- added U$1: PIN_3X8, pinhead_3row:PIN_3X8
- IC3: value 74ALS00N -> 74LS32N; device 74xx-us:74ALS00N -> 74xx-us:74LS32N
Connections:
- net -ADDR-REG-LD0 renamed -ADDR-REG-ID1
- net -ADDR-REG-LD1 renamed -ADDR-REG-ID3
- net -ADDR-REG-RD0 renamed -ADDR-REG-ID0
- net -ADDR-REG-RD1 renamed -ADDR-REG-ID2
- removed net -ROME000: IC10D.I0, IC7A.Y6
- removed net -ROMF000: IC10D.I1, IC7A.Y7
- new net -TMP-REG-RD: IC25A.G
- new net -TMP-REG-WR: IC25B.G
- new net -TREG-LD0: IC25B.Y0
- new net -TREG-LD1: IC14D.I, IC25B.Y1
- new net -TREG-LD2: IC14F.I, IC25B.Y2
- new net -TREG-LD3: IC14A.I, IC25B.Y3
- new net -TREG-LDO: IC14C.I
- new net -TREG-RD0: IC15A.OC, IC16A.OC, IC25A.Y0
- new net -TREG-RD1: IC17A.OC, IC19A.OC, IC25A.Y1
- new net -TREG-RD2: IC21A.OC, IC22A.OC, IC25A.Y2
- new net -TREG-RD3: IC23A.OC, IC24A.OC, IC25A.Y3
- new net N$21: IC14C.O, IC15A.CLK, IC16A.CLK
- new net N$23: IC14D.O, IC17A.CLK, IC19A.CLK
- new net N$24: IC7A.G2B, JP1.2
- new net N$25: IC10D.I0, IC10D.I1, IC3A.O
- new net N$26: IC4A.I6, RN8.8, U$1.23
- new net N$27: IC4A.I7, RN8.9, U$1.24
- new net N$28: IC18A.I7, RN7.9, U$1.1
- new net N$29: IC18A.I6, RN7.8, U$1.2
- new net N$30: IC18A.I5, RN7.7, U$1.3
- new net N$31: IC18A.I4, RN7.6, U$1.4
- new net N$32: IC18A.I0, RN7.2, U$1.8
- new net N$34: IC18A.I1, RN7.3, U$1.7
- new net N$35: IC18A.I2, RN7.4, U$1.6
- new net N$36: IC7A.Y7, U$1.16
- new net N$37: IC7A.Y6, U$1.15
- new net N$38: IC7A.Y5, U$1.14
- new net N$39: IC7A.Y4, U$1.13
- new net N$40: IC7A.Y3, U$1.12
- new net N$41: IC7A.Y2, U$1.11
- new net N$42: IC7A.Y1, U$1.10
- new net N$43: IC7A.Y0, U$1.9
- new net N$44: IC18A.I3, RN7.5, U$1.5
- new net N$45: IC14F.O, IC21A.CLK, IC22A.CLK
- new net N$46: IC14A.O, IC23A.CLK, IC24A.CLK
- new net TMP-ID0: IC25A.A, IC25B.A
- new net TMP-ID1: IC25A.B, IC25B.B
- net -BUS-EN: now also IC3A.I1, JP1.1
- net -VMA: now also IC14E.I, IC3A.I0; no longer IC10C.I0, IC10C.I1, IC3B.I0, IC3B.I1
- net ADDR15: now also IC10B.I0; no longer IC3A.I0
- net BADDR0: no longer RN1-1.1
- net BADDR1: no longer RN1-2.1
- net BADDR10: no longer RN2-3.1
- net BADDR11: no longer RN2-4.1
- net BADDR12: no longer RN2-5.1
- net BADDR13: no longer RN2-6.1
- net BADDR14: no longer RN2-7.1
- net BADDR15: now also IC14B.I; no longer IC10B.I0, IC10B.I1, RN2-8.1
- net BADDR2: no longer RN1-3.1
- net BADDR3: no longer RN1-4.1
- net BADDR4: no longer RN1-5.1
- net BADDR5: no longer RN1-6.1
- net BADDR6: no longer RN1-7.1
- net BADDR7: no longer RN1-8.1
- net BADDR8: no longer RN2-1.1
- net BADDR9: no longer RN2-2.1
- net BDATA0: no longer RN4-1.1
- net BDATA1: no longer RN4-2.1
- net BDATA2: no longer RN4-3.1
- net BDATA3: no longer RN4-4.1
- net BDATA4: no longer RN4-5.1
- net BDATA5: no longer RN4-6.1
- net BDATA6: no longer RN4-7.1
- net BDATA7: no longer RN4-8.1
- net DATA0: now also IC15A.1D, IC15A.1Q, IC17A.1D, IC17A.1Q, IC21A.1D, IC21A.1Q, IC23A.1D, IC23A.1Q; no longer RN3-1.1
- net DATA1: now also IC15A.2D, IC15A.2Q, IC17A.2D, IC17A.2Q, IC21A.2D, IC21A.2Q, IC23A.2D, IC23A.2Q; no longer RN3-2.1
- net DATA10: now also IC16A.3D, IC16A.3Q, IC19A.3D, IC19A.3Q, IC22A.3D, IC22A.3Q, IC24A.3D, IC24A.3Q
- net DATA11: now also IC16A.4D, IC16A.4Q, IC19A.4D, IC19A.4Q, IC22A.4D, IC22A.4Q, IC24A.4D, IC24A.4Q
- net DATA12: now also IC16A.5D, IC16A.5Q, IC19A.5D, IC19A.5Q, IC22A.5D, IC22A.5Q, IC24A.5D, IC24A.5Q
- net DATA13: now also IC16A.6D, IC16A.6Q, IC19A.6D, IC19A.6Q, IC22A.6D, IC22A.6Q, IC24A.6D, IC24A.6Q
- net DATA14: now also IC16A.7D, IC16A.7Q, IC19A.7D, IC19A.7Q, IC22A.7D, IC22A.7Q, IC24A.7D, IC24A.7Q
- net DATA15: now also IC16A.8D, IC16A.8Q, IC19A.8D, IC19A.8Q, IC22A.8D, IC22A.8Q, IC24A.8D, IC24A.8Q
- net DATA2: now also IC15A.3D, IC15A.3Q, IC17A.3D, IC17A.3Q, IC21A.3D, IC21A.3Q, IC23A.3D, IC23A.3Q; no longer RN3-3.1
- net DATA3: now also IC15A.4D, IC15A.4Q, IC17A.4D, IC17A.4Q, IC21A.4D, IC21A.4Q, IC23A.4D, IC23A.4Q; no longer RN3-4.1
- net DATA4: now also IC15A.5D, IC15A.5Q, IC17A.5D, IC17A.5Q, IC21A.5D, IC21A.5Q, IC23A.5D, IC23A.5Q; no longer RN3-5.1
- net DATA5: now also IC15A.6D, IC15A.6Q, IC17A.6D, IC17A.6Q, IC21A.6D, IC21A.6Q, IC23A.6D, IC23A.6Q; no longer RN3-6.1
- net DATA6: now also IC15A.7D, IC15A.7Q, IC17A.7D, IC17A.7Q, IC21A.7D, IC21A.7Q, IC23A.7D, IC23A.7Q; no longer RN3-7.1
- net DATA7: now also IC15A.8D, IC15A.8Q, IC17A.8D, IC17A.8Q, IC21A.8D, IC21A.8Q, IC23A.8D, IC23A.8Q; no longer RN3-8.1
- net DATA8: now also IC16A.1D, IC16A.1Q, IC19A.1D, IC19A.1Q, IC22A.1D, IC22A.1Q, IC24A.1D, IC24A.1Q
- net DATA9: now also IC16A.2D, IC16A.2Q, IC19A.2D, IC19A.2Q, IC22A.2D, IC22A.2Q, IC24A.2D, IC24A.2Q
- net GND: now also C14.2, C15.2, C16.2, C17.2, C18.2, C19.1, C20.1, C21.1, C22.1, C23.1, C24.1, IC3B.I0, IC3B.I1, IC3D.I0, IC3D.I1, JP1.3; no longer IC7A.G2B
- net N$1: now also IC18A.O; no longer IC10D.O
- net N$10: now also IC4A.I5, RN8.7, U$1.22; no longer IC4A.I1, IC7A.Y0
- net N$12: now also IC14E.O; no longer IC10C.O
- net N$13: now also IC14B.O; no longer IC10B.O
- net N$19: now also IC10C.O; no longer IC3D.O
- net N$20: now also IC10B.O, IC10C.I0, IC10C.I1; no longer IC3A.O, IC3D.I0, IC3D.I1
- net N$22: now also IC10B.I1, IC10D.O; no longer IC3A.I1, IC3B.O
- net N$5: now also IC4A.I0, RN8.2, U$1.17; no longer IC4A.I6, IC7A.Y5
- net N$6: now also IC4A.I1, RN8.3, U$1.18; no longer IC4A.I5, IC7A.Y4
- net N$7: now also IC4A.I2, RN8.4, U$1.19; no longer IC4A.I4, IC7A.Y3
- net N$8: now also RN8.5, U$1.20; no longer IC7A.Y2
- net N$9: now also IC4A.I4, RN8.6, U$1.21; no longer IC4A.I2, IC7A.Y1
- net VCC: now also C14.1, C15.1, C16.1, C17.1, C18.1, C19.2, C20.2, C21.2, C22.2, C23.2, C24.2, RN7.1, RN8.1; no longer IC4A.I0, IC4A.I7, RN1_.1, RN2_.1, RN3_.1, RN4_.1
Other:
- note removed: "Optional - Leave empty"

Commit message: cleaning up paths
Parts:
- removed IC15, IC16, IC17, IC19, IC21, IC22, IC23, IC24: 74LS374N, 74xx-us:74LS374N
- removed IC25: 74LS139N, 74xx-us:74LS139N
- added IC26, IC27, IC28, IC29: 74LS374N, 74xx-us:74LS374N
- added RN5, RN6: (no value), resistor-net:RNX8
Connections:
- removed net -TMP-REG-RD: IC25A.G
- removed net -TMP-REG-WR: IC25B.G
- removed net -TREG-LD0: IC25B.Y0
- removed net -TREG-LD1: IC14D.I, IC25B.Y1
- removed net -TREG-LD2: IC14F.I, IC25B.Y2
- removed net -TREG-LD3: IC14A.I, IC25B.Y3
- removed net -TREG-LDO: IC14C.I
- removed net -TREG-RD0: IC15A.OC, IC16A.OC, IC25A.Y0
- removed net -TREG-RD1: IC17A.OC, IC19A.OC, IC25A.Y1
- removed net -TREG-RD2: IC21A.OC, IC22A.OC, IC25A.Y2
- removed net -TREG-RD3: IC23A.OC, IC24A.OC, IC25A.Y3
- removed net N$21: IC14C.O, IC15A.CLK, IC16A.CLK
- removed net N$23: IC14D.O, IC17A.CLK, IC19A.CLK
- removed net N$45: IC14F.O, IC21A.CLK, IC22A.CLK
- removed net N$46: IC14A.O, IC23A.CLK, IC24A.CLK
- removed net TMP-ID0: IC25A.A, IC25B.A
- removed net TMP-ID1: IC25A.B, IC25B.B
- new net N$33: IC14A.O, IC26A.CLK, IC27A.CLK
- new net N$47: IC14F.O, IC28A.CLK, IC29A.CLK
- net -TMP-REG-LD0: now also IC14A.I
- net -TMP-REG-LD1: now also IC14F.I
- net -TMP-REG-RD0: now also IC26A.OC, IC27A.OC
- net -TMP-REG-RD1: now also IC28A.OC, IC29A.OC
- net DATA0: now also IC26A.1D, IC26A.1Q, IC28A.1D, IC28A.1Q, RN5-1.1; no longer IC15A.1D, IC15A.1Q, IC17A.1D, IC17A.1Q, IC21A.1D, IC21A.1Q, IC23A.1D, IC23A.1Q
- net DATA1: now also IC26A.2D, IC26A.2Q, IC28A.2D, IC28A.2Q, RN5-2.1; no longer IC15A.2D, IC15A.2Q, IC17A.2D, IC17A.2Q, IC21A.2D, IC21A.2Q, IC23A.2D, IC23A.2Q
- net DATA10: now also IC27A.3D, IC27A.3Q, IC29A.3D, IC29A.3Q, RN6-3.1; no longer IC16A.3D, IC16A.3Q, IC19A.3D, IC19A.3Q, IC22A.3D, IC22A.3Q, IC24A.3D, IC24A.3Q
- net DATA11: now also IC27A.4D, IC27A.4Q, IC29A.4D, IC29A.4Q, RN6-4.1; no longer IC16A.4D, IC16A.4Q, IC19A.4D, IC19A.4Q, IC22A.4D, IC22A.4Q, IC24A.4D, IC24A.4Q
- net DATA12: now also IC27A.5D, IC27A.5Q, IC29A.5D, IC29A.5Q, RN6-5.1; no longer IC16A.5D, IC16A.5Q, IC19A.5D, IC19A.5Q, IC22A.5D, IC22A.5Q, IC24A.5D, IC24A.5Q
- net DATA13: now also IC27A.6D, IC27A.6Q, IC29A.6D, IC29A.6Q, RN6-6.1; no longer IC16A.6D, IC16A.6Q, IC19A.6D, IC19A.6Q, IC22A.6D, IC22A.6Q, IC24A.6D, IC24A.6Q
- net DATA14: now also IC27A.7D, IC27A.7Q, IC29A.7D, IC29A.7Q, RN6-7.1; no longer IC16A.7D, IC16A.7Q, IC19A.7D, IC19A.7Q, IC22A.7D, IC22A.7Q, IC24A.7D, IC24A.7Q
- net DATA15: now also IC27A.8D, IC27A.8Q, IC29A.8D, IC29A.8Q, RN6-8.1; no longer IC16A.8D, IC16A.8Q, IC19A.8D, IC19A.8Q, IC22A.8D, IC22A.8Q, IC24A.8D, IC24A.8Q
- net DATA2: now also IC26A.3D, IC26A.3Q, IC28A.3D, IC28A.3Q, RN5-3.1; no longer IC15A.3D, IC15A.3Q, IC17A.3D, IC17A.3Q, IC21A.3D, IC21A.3Q, IC23A.3D, IC23A.3Q
- net DATA3: now also IC26A.4D, IC26A.4Q, IC28A.4D, IC28A.4Q, RN5-4.1; no longer IC15A.4D, IC15A.4Q, IC17A.4D, IC17A.4Q, IC21A.4D, IC21A.4Q, IC23A.4D, IC23A.4Q
- net DATA4: now also IC26A.5D, IC26A.5Q, IC28A.5D, IC28A.5Q, RN5-5.1; no longer IC15A.5D, IC15A.5Q, IC17A.5D, IC17A.5Q, IC21A.5D, IC21A.5Q, IC23A.5D, IC23A.5Q
- net DATA5: now also IC26A.6D, IC26A.6Q, IC28A.6D, IC28A.6Q, RN5-6.1; no longer IC15A.6D, IC15A.6Q, IC17A.6D, IC17A.6Q, IC21A.6D, IC21A.6Q, IC23A.6D, IC23A.6Q
- net DATA6: now also IC26A.7D, IC26A.7Q, IC28A.7D, IC28A.7Q, RN5-7.1; no longer IC15A.7D, IC15A.7Q, IC17A.7D, IC17A.7Q, IC21A.7D, IC21A.7Q, IC23A.7D, IC23A.7Q
- net DATA7: now also IC26A.8D, IC26A.8Q, IC28A.8D, IC28A.8Q, RN5-8.1; no longer IC15A.8D, IC15A.8Q, IC17A.8D, IC17A.8Q, IC21A.8D, IC21A.8Q, IC23A.8D, IC23A.8Q
- net DATA8: now also IC27A.1D, IC27A.1Q, IC29A.1D, IC29A.1Q, RN6-1.1; no longer IC16A.1D, IC16A.1Q, IC19A.1D, IC19A.1Q, IC22A.1D, IC22A.1Q, IC24A.1D, IC24A.1Q
- net DATA9: now also IC27A.2D, IC27A.2Q, IC29A.2D, IC29A.2Q, RN6-2.1; no longer IC16A.2D, IC16A.2Q, IC19A.2D, IC19A.2Q, IC22A.2D, IC22A.2Q, IC24A.2D, IC24A.2Q
- net GND: now also RN5_.1, RN6_.1
